Commit message: 260130.0200AM

File: src/my_amr_description/urdf/mobile_base.xacro (robot description, xacro)
@@ -58,5 +58,5 @@
                     <origin xyz="0 0 ${b/2.0}" rpy="0 0 0"/>
                 </collision>
-                <xacro:box_inertia m="${body_mass}" l="${c}" w="${c}" h="${b}"
+                <xacro:box_inertia m="${body_mass}" l="${2*c}" w="${2*c}" h="${2*b}"
                                    xyz="0 0 ${b/2.0}" rpy="0 0 0"/>
             </link>
@@ -66,4 +66,7 @@
                 <origin xyz="0 0 ${2.0*r_caster}" rpy="0 0 0"/>
             </joint>
+            <gazebo reference="base_link">
+                <material>Gazebo/Orange</material>
+            </gazebo>
         <!-- Lidar -->
             <link name="lidar_link">
@@ -81,5 +84,5 @@
                     <origin xyz="0 0 ${(lidar_length + roof_height)/2.0}" rpy="0 0 0"/>
                 </collision>
-                <xacro:cylinder_inertia m="${lidar_mass}" r="${lidar_radius}" h="${lidar_length}"
+                <xacro:cylinder_inertia m="${lidar_mass}" r="${2*lidar_radius}" h="${2*lidar_length}"
                                         xyz="0 0 ${(lidar_length + roof_height)/2.0}" rpy="0 0 0"/>
             </link>
@@ -89,4 +92,7 @@
                 <origin xyz="0 0 ${b}" rpy="0 0 0"/>
             </joint>
+            <gazebo reference="lidar_link">
+                <material>Gazebo/Black</material>
+            </gazebo>
         <!-- Wheels -->
             <xacro:macro name="wheel_link" params="prefix offset y">
@@ -105,5 +111,5 @@
                         <origin xyz="0 ${offset} 0" rpy="${pi/2.0} 0 0"/>
                     </collision>
-                    <xacro:cylinder_inertia m="${wheel_mass}" r="${r}" h="${d}"
+                    <xacro:cylinder_inertia m="${wheel_mass}" r="${2*r}" h="${2*d}"
                                             xyz="0 ${offset} 0" rpy="${pi/2.0} 0 0"/>
                 </link>
@@ -114,4 +120,7 @@
                     <axis xyz="0 1 0"/>
                 </joint>
+                <gazebo reference="${prefix}_wheel_link">
+                    <material>Gazebo/Grey</material>
+                </gazebo>
             </xacro:macro>
             <xacro:wheel_link prefix="right" offset="${wheel_offset}" y="${-S4}"/>
@@ -133,5 +142,5 @@
                         <origin xyz="0 0 0" rpy="0 0 0"/>
                     </collision>
-                    <xacro:sphere_inertia m="${caster_mass}" r="${r_caster}"
+                    <xacro:sphere_inertia m="${caster_mass}" r="${2*r_caster}"
                                           xyz="0 0 0" rpy="0 0 0"/>
                 </link>
@@ -141,4 +150,7 @@
                     <origin xyz="${x} ${y} ${-r_caster}" rpy="0 0 0"/>
                 </joint>
+                <gazebo reference="caster_wheel_${id}_link">
+                    <material>Gazebo/Black</material>
+                </gazebo>
             </xacro:macro>
             <xacro:caster_wheel_link id="1" x="${-S2}" y="${S3}"/>
@@ -161,5 +173,5 @@
                     <origin xyz="0 0 ${roof_height/2.0}" rpy="0 0 0"/>
                 </collision>
-                <xacro:box_inertia m="${roof_mass}" l="${c}" w="${c}" h="${roof_height}"
+                <xacro:box_inertia m="${roof_mass}" l="${2*c}" w="${2*c}" h="${2*roof_height}"
                                    xyz="0 0 ${roof_height/2.0}" rpy="0 0 0"/>
             </link>
@@ -169,3 +181,6 @@
                 <origin xyz="0 0 ${b}" rpy="0 0 0"/>
             </joint>
+            <gazebo reference="roof_link">
+                <material>Gazebo/Blue</material>
+            </gazebo>
 </robot>

File: src/my_amr_description/urdf/my_amr.urdf.xacro (robot description, xacro)
@@ -3,3 +3,4 @@
     <xacro:include filename="common_properties.xacro"/>
     <xacro:include filename="mobile_base.xacro"/>
+    <xacro:include filename="mobile_base_gazebo.xacro"/>
 </robot>

Commit message: 260130.0535PM

File: src/my_amr_description/urdf/mobile_base.xacro (robot description, xacro)
@@ -49,5 +49,5 @@
                         <box size="${c} ${c} ${b}"/>
                     </geometry>
-                    <origin xyz="0 0 ${b/2.0}" rpy="0 0 0"/>
+                    <origin xyz="0 0 ${S1}" rpy="0 0 0"/>
                     <material name="orange"/>
                 </visual>
@@ -56,13 +56,13 @@
                         <box size="${c} ${c} ${b}"/>
                     </geometry>
-                    <origin xyz="0 0 ${b/2.0}" rpy="0 0 0"/>
+                    <origin xyz="0 0 ${S1}" rpy="0 0 0"/>
                 </collision>
-                <xacro:box_inertia m="${body_mass}" l="${2*c}" w="${2*c}" h="${2*b}"
-                                   xyz="0 0 ${b/2.0}" rpy="0 0 0"/>
+                <xacro:box_inertia m="${body_mass}" l="${c}" w="${c}" h="${b}"
+                                   xyz="0 0 ${S1}" rpy="0 0 0"/>
             </link>
             <joint name="base_footprint_base_joint" type="fixed">
                 <parent link="base_footprint"/>
                 <child link="base_link"/>
-                <origin xyz="0 0 ${2.0*r_caster}" rpy="0 0 0"/>
+                <origin xyz="0 0 0" rpy="0 0 0"/>
             </joint>
             <gazebo reference="base_link">
@@ -84,5 +84,5 @@
                     <origin xyz="0 0 ${(lidar_length + roof_height)/2.0}" rpy="0 0 0"/>
                 </collision>
-                <xacro:cylinder_inertia m="${lidar_mass}" r="${2*lidar_radius}" h="${2*lidar_length}"
+                <xacro:cylinder_inertia m="${lidar_mass}" r="${lidar_radius}" h="${lidar_length}"
                                         xyz="0 0 ${(lidar_length + roof_height)/2.0}" rpy="0 0 0"/>
             </link>
@@ -90,5 +90,5 @@
                 <parent link="base_link"/>
                 <child link="lidar_link"/>
-                <origin xyz="0 0 ${b}" rpy="0 0 0"/>
+                <origin xyz="0 0 ${S1 + (b + 2*r_caster - S1)}" rpy="0 0 0"/>
             </joint>
             <gazebo reference="lidar_link">
@@ -111,5 +111,5 @@
                         <origin xyz="0 ${offset} 0" rpy="${pi/2.0} 0 0"/>
                     </collision>
-                    <xacro:cylinder_inertia m="${wheel_mass}" r="${2*r}" h="${2*d}"
+                    <xacro:cylinder_inertia m="${wheel_mass}" r="${r}" h="${d}"
                                             xyz="0 ${offset} 0" rpy="${pi/2.0} 0 0"/>
                 </link>
@@ -117,5 +117,5 @@
                     <parent link="base_link"/>
                     <child link="${prefix}_wheel_link"/>
-                    <origin xyz="0 ${y} ${r - 2.0*r_caster}" rpy="0 0 0"/>
+                    <origin xyz="0 ${y} ${r}" rpy="0 0 0"/>
                     <axis xyz="0 1 0"/>
                 </joint>
@@ -142,5 +142,5 @@
                         <origin xyz="0 0 0" rpy="0 0 0"/>
                     </collision>
-                    <xacro:sphere_inertia m="${caster_mass}" r="${2*r_caster}"
+                    <xacro:sphere_inertia m="${caster_mass}" r="${r_caster}"
                                           xyz="0 0 0" rpy="0 0 0"/>
                 </link>
@@ -148,8 +148,10 @@
                     <parent link="base_link"/>
                     <child link="caster_wheel_${id}_link"/>
-                    <origin xyz="${x} ${y} ${-r_caster}" rpy="0 0 0"/>
+                    <origin xyz="${x} ${y} ${r_caster}" rpy="0 0 0"/>
                 </joint>
                 <gazebo reference="caster_wheel_${id}_link">
                     <material>Gazebo/Black</material>
+                    <mu1 value="0.1"/>
+                    <mu2 value="0.1"/>
                 </gazebo>
             </xacro:macro>
@@ -173,5 +175,5 @@
                     <origin xyz="0 0 ${roof_height/2.0}" rpy="0 0 0"/>
                 </collision>
-                <xacro:box_inertia m="${roof_mass}" l="${2*c}" w="${2*c}" h="${2*roof_height}"
+                <xacro:box_inertia m="${roof_mass}" l="${c}" w="${c}" h="${roof_height}"
                                    xyz="0 0 ${roof_height/2.0}" rpy="0 0 0"/>
             </link>
@@ -179,5 +181,5 @@
                 <parent link="base_link"/>
                 <child link="roof_link"/>
-                <origin xyz="0 0 ${b}" rpy="0 0 0"/>
+                <origin xyz="0 0 ${S1 + (b + 2*r_caster - S1)}" rpy="0 0 0"/>
             </joint>
             <gazebo reference="roof_link">
