Commit message: 260130.0055AM - update inertia and collision in urdf

File: src/my_amr_description/urdf/common_properties.xacro (robot description, xacro)
@@ -1,15 +1,44 @@
 <?xml version="1.0"?>
 <robot name="my_amr" xmlns:xacro="http://www.ros.org/wiki/xacro">
-    <material name="orange">
-        <color rgba="1 0.3 0 1"/>
-    </material>
-    <material name="blue">
-        <color rgba="0 0 0.5 1"/>
-    </material>
-    <material name="black">
-        <color rgba="0 0 0 1"/>
-    </material>
-    <material name="grey">
-        <color rgba="0.5 0.5 0.5 1"/>
-    </material>
+    <!-- Colors -->
+        <material name="orange">
+            <color rgba="1 0.3 0 1"/>
+        </material>
+        <material name="blue">
+            <color rgba="0 0 0.5 1"/>
+        </material>
+        <material name="black">
+            <color rgba="0 0 0 1"/>
+        </material>
+        <material name="grey">
+            <color rgba="0.5 0.5 0.5 1"/>
+        </material>
+    <!-- Inertia -->
+        <xacro:macro name="box_inertia" params="m l w h xyz rpy">
+            <inertial>
+                <origin xyz="${xyz}" rpy="${rpy}"/>
+                <mass value="${m}"/>
+                <inertia ixx="${(m/12.0) * (h*h + l*l)}" ixy="0" ixz="0"
+                         iyy="${(m/12.0) * (w*w + l*l)}" iyz="0"
+                         izz="${(m/12.0) * (w*w + h*h)}"/>
+            </inertial>
+        </xacro:macro>
+        <xacro:macro name="cylinder_inertia" params="m r h xyz rpy">
+            <inertial>
+                <origin xyz="${xyz}" rpy="${rpy}"/>
+                <mass value="${m}"/>
+                <inertia ixx="${(m/12.0) * (3.0*r*r + h*h)}" ixy="0" ixz="0"
+                         iyy="${(m/12.0) * (3.0*r*r + h*h)}" iyz="0"
+                         izz="${(m/2.0) * (r*r)}"/>
+            </inertial>
+        </xacro:macro>
+        <xacro:macro name="sphere_inertia" params="m r xyz rpy">
+            <inertial>
+                <origin xyz="${xyz}" rpy="${rpy}"/>
+                <mass value="${m}"/>
+                <inertia ixx="${(2/5) * m * r * r}" ixy="0" ixz="0"
+                         iyy="${(2/5) * m * r * r}" iyz="0"
+                         izz="${(2/5) * m * r * r}"/>
+            </inertial>
+        </xacro:macro>
 </robot>

File: src/my_amr_description/urdf/mobile_base.xacro (robot description, xacro)
@@ -7,4 +7,6 @@
             <!-- Body Height -->
             <xacro:property name="b" value="0.1"/>
+            <!-- Body Mass -->
+            <xacro:property name="body_mass" value="20.0"/>
         <!-- Wheel and caster dimensions -->
             <!-- Wheel radius -->
@@ -14,6 +16,10 @@
             <!-- Wheel offset -->
                 <xacro:property name="wheel_offset" value="0.01"/>
+            <!-- Wheel Mass -->
+                <xacro:property name="wheel_mass" value="0.5"/>
             <!-- Caster radius -->
                 <xacro:property name="r_caster" value="0.02"/>
+            <!-- Caster Mass -->
+                <xacro:property name="caster_mass" value="0.1"/>
         <!-- Lidar and roof dimensions -->
             <!-- Lidar Radius -->
@@ -21,11 +27,15 @@
             <!-- Lidar Length -->
                 <xacro:property name="lidar_length" value="0.05"/>
+            <!-- Lidar Mass -->
+                <xacro:property name="lidar_mass" value="0.5"/>
             <!-- Roof Height-->
                 <xacro:property name="roof_height" value="0.001"/>
+            <!-- Roof Mass -->
+                <xacro:property name="roof_mass" value="1.0"/>
         <!-- S Value -->
-            <xacro:property name="S1" value="${b/2+2*r_caster}"/>
+            <xacro:property name="S1" value="${b/2.0+2.0*r_caster}"/>
             <xacro:property name="S2" value="0.2"/>
             <xacro:property name="S3" value="0.125"/>
-            <xacro:property name="S4" value="${c/2-d/2}"/>
+            <xacro:property name="S4" value="${c/2.0-d/2.0}"/>
     <!-- Links -->
         <!-- Base Footprint -->
@@ -39,12 +49,20 @@
                         <box size="${c} ${c} ${b}"/>
                     </geometry>
-                    <origin xyz="0 0 ${b/2}" rpy="0 0 0"/>
+                    <origin xyz="0 0 ${b/2.0}" rpy="0 0 0"/>
                     <material name="orange"/>
                 </visual>
+                <collision>
+                    <geometry>
+                        <box size="${c} ${c} ${b}"/>
+                    </geometry>
+                    <origin xyz="0 0 ${b/2.0}" rpy="0 0 0"/>
+                </collision>
+                <xacro:box_inertia m="${body_mass}" l="${c}" w="${c}" h="${b}"
+                                   xyz="0 0 ${b/2.0}" rpy="0 0 0"/>
             </link>
             <joint name="base_footprint_base_joint" type="fixed">
                 <parent link="base_footprint"/>
                 <child link="base_link"/>
-                <origin xyz="0 0 ${2*r_caster}" rpy="0 0 0"/>
+                <origin xyz="0 0 ${2.0*r_caster}" rpy="0 0 0"/>
             </joint>
         <!-- Lidar -->
@@ -54,7 +72,15 @@
                         <cylinder radius="${lidar_radius}" length="${lidar_length}"/>
                     </geometry>
-                    <origin xyz="0 0 ${(lidar_length + roof_height)/2}" rpy="0 0 0"/>
+                    <origin xyz="0 0 ${(lidar_length + roof_height)/2.0}" rpy="0 0 0"/>
                     <material name="black"/>
                 </visual>
+                <collision>
+                    <geometry>
+                        <cylinder radius="${lidar_radius}" length="${lidar_length}"/>
+                    </geometry>
+                    <origin xyz="0 0 ${(lidar_length + roof_height)/2.0}" rpy="0 0 0"/>
+                </collision>
+                <xacro:cylinder_inertia m="${lidar_mass}" r="${lidar_radius}" h="${lidar_length}"
+                                        xyz="0 0 ${(lidar_length + roof_height)/2.0}" rpy="0 0 0"/>
             </link>
             <joint name="base_lidar_joint" type="fixed">
@@ -73,9 +99,17 @@
                         <material name="grey"/>
                     </visual>
+                    <collision>
+                        <geometry>
+                            <cylinder radius="${r}" length="${d}"/>
+                        </geometry>
+                        <origin xyz="0 ${offset} 0" rpy="${pi/2.0} 0 0"/>
+                    </collision>
+                    <xacro:cylinder_inertia m="${wheel_mass}" r="${r}" h="${d}"
+                                            xyz="0 ${offset} 0" rpy="${pi/2.0} 0 0"/>
                 </link>
                 <joint name="base_${prefix}_wheel_joint" type="continuous">
                     <parent link="base_link"/>
                     <child link="${prefix}_wheel_link"/>
-                    <origin xyz="0 ${y} ${r - 2*r_caster}" rpy="0 0 0"/>
+                    <origin xyz="0 ${y} ${r - 2.0*r_caster}" rpy="0 0 0"/>
                     <axis xyz="0 1 0"/>
                 </joint>
@@ -93,4 +127,12 @@
                         <material name="black"/>
                     </visual>
+                    <collision>
+                        <geometry>
+                            <sphere radius="${r_caster}"/>
+                        </geometry>
+                        <origin xyz="0 0 0" rpy="0 0 0"/>
+                    </collision>
+                    <xacro:sphere_inertia m="${caster_mass}" r="${r_caster}"
+                                          xyz="0 0 0" rpy="0 0 0"/>
                 </link>
                 <joint name="base_caster_wheel_${id}_joint" type="fixed">
@@ -110,7 +152,15 @@
                         <box size="${c} ${c} ${roof_height}"/>
                     </geometry>
-                    <origin xyz="0 0 ${roof_height/2}" rpy="0 0 0"/>
+                    <origin xyz="0 0 ${roof_height/2.0}" rpy="0 0 0"/>
                     <material name="blue"/>
                 </visual>
+                <collision>
+                    <geometry>
+                        <box size="${c} ${c} ${roof_height}"/>
+                    </geometry>
+                    <origin xyz="0 0 ${roof_height/2.0}" rpy="0 0 0"/>
+                </collision>
+                <xacro:box_inertia m="${roof_mass}" l="${c}" w="${c}" h="${roof_height}"
+                                   xyz="0 0 ${roof_height/2.0}" rpy="0 0 0"/>
             </link>
             <joint name="base_roof_joint" type="fixed">

Commit message: 260131.0620PM - Added Lidar sensor

File: src/my_amr_description/urdf/common_properties.xacro (robot description, xacro)
@@ -2,5 +2,5 @@
 <robot name="my_amr" xmlns:xacro="http://www.ros.org/wiki/xacro">
     <!-- Colors -->
-        <material name="orange">
+        <material name="red">
             <color rgba="1 0.3 0 1"/>
         </material>
@@ -14,4 +14,41 @@
             <color rgba="0.5 0.5 0.5 1"/>
         </material>
+    <!-- Variables and Constants -->
+        <!-- Body dimensions -->
+            <!-- Body Width/Length -->
+            <xacro:property name="c" value="0.5"/>
+            <!-- Body Height -->
+            <xacro:property name="b" value="0.1"/>
+            <!-- Body Mass -->
+            <xacro:property name="body_mass" value="20.0"/>
+        <!-- Wheel and caster dimensions -->
+            <!-- Wheel radius -->
+                <xacro:property name="r" value="0.05"/>
+            <!-- Wheel width -->
+                <xacro:property name="d" value="0.02"/>
+            <!-- Wheel offset -->
+                <xacro:property name="wheel_offset" value="0.01"/>
+            <!-- Wheel Mass -->
+                <xacro:property name="wheel_mass" value="0.5"/>
+            <!-- Caster radius -->
+                <xacro:property name="r_caster" value="0.02"/>
+            <!-- Caster Mass -->
+                <xacro:property name="caster_mass" value="0.1"/>
+        <!-- Lidar and Roof dimensions -->
+            <!-- Lidar Radius -->
+                <xacro:property name="lidar_radius" value="0.05"/>
+            <!-- Lidar Length -->
+                <xacro:property name="lidar_length" value="0.05"/>
+            <!-- Lidar Mass -->
+                <xacro:property name="lidar_mass" value="0.5"/>
+            <!-- Roof Height-->
+                <xacro:property name="roof_height" value="0.001"/>
+            <!-- Roof Mass -->
+                <xacro:property name="roof_mass" value="1.0"/>
+        <!-- S Value -->
+            <xacro:property name="S1" value="${b/2.0+2.0*r_caster}"/>
+            <xacro:property name="S2" value="0.2"/>
+            <xacro:property name="S3" value="0.125"/>
+            <xacro:property name="S4" value="${c/2.0-d/2.0}"/>
     <!-- Inertia -->
         <xacro:macro name="box_inertia" params="m l w h xyz rpy">

File: src/my_amr_description/urdf/mobile_base.xacro (robot description, xacro)
@@ -1,41 +1,4 @@
 <?xml version="1.0"?>
 <robot name="my_amr" xmlns:xacro="http://www.ros.org/wiki/xacro">
-    <!-- Variables and Constants -->
-        <!-- Body dimensions -->
-            <!-- Body Width/Length -->
-            <xacro:property name="c" value="0.5"/>
-            <!-- Body Height -->
-            <xacro:property name="b" value="0.1"/>
-            <!-- Body Mass -->
-            <xacro:property name="body_mass" value="20.0"/>
-        <!-- Wheel and caster dimensions -->
-            <!-- Wheel radius -->
-                <xacro:property name="r" value="0.05"/>
-            <!-- Wheel width -->
-                <xacro:property name="d" value="0.02"/>
-            <!-- Wheel offset -->
-                <xacro:property name="wheel_offset" value="0.01"/>
-            <!-- Wheel Mass -->
-                <xacro:property name="wheel_mass" value="0.5"/>
-            <!-- Caster radius -->
-                <xacro:property name="r_caster" value="0.02"/>
-            <!-- Caster Mass -->
-                <xacro:property name="caster_mass" value="0.1"/>
-        <!-- Lidar and roof dimensions -->
-            <!-- Lidar Radius -->
-                <xacro:property name="lidar_radius" value="0.05"/>
-            <!-- Lidar Length -->
-                <xacro:property name="lidar_length" value="0.05"/>
-            <!-- Lidar Mass -->
-                <xacro:property name="lidar_mass" value="0.5"/>
-            <!-- Roof Height-->
-                <xacro:property name="roof_height" value="0.001"/>
-            <!-- Roof Mass -->
-                <xacro:property name="roof_mass" value="1.0"/>
-        <!-- S Value -->
-            <xacro:property name="S1" value="${b/2.0+2.0*r_caster}"/>
-            <xacro:property name="S2" value="0.2"/>
-            <xacro:property name="S3" value="0.125"/>
-            <xacro:property name="S4" value="${c/2.0-d/2.0}"/>
     <!-- Links -->
         <!-- Base Footprint -->
@@ -50,5 +13,5 @@
                     </geometry>
                     <origin xyz="0 0 ${S1}" rpy="0 0 0"/>
-                    <material name="orange"/>
+                    <material name="red"/>
                 </visual>
                 <collision>
@@ -67,31 +30,5 @@
             </joint>
             <gazebo reference="base_link">
-                <material>Gazebo/Orange</material>
-            </gazebo>
-        <!-- Lidar -->
-            <link name="lidar_link">
-                <visual>
-                    <geometry>
-                        <cylinder radius="${lidar_radius}" length="${lidar_length}"/>
-                    </geometry>
-                    <origin xyz="0 0 ${(lidar_length + roof_height)/2.0}" rpy="0 0 0"/>
-                    <material name="black"/>
-                </visual>
-                <collision>
-                    <geometry>
-                        <cylinder radius="${lidar_radius}" length="${lidar_length}"/>
-                    </geometry>
-                    <origin xyz="0 0 ${(lidar_length + roof_height)/2.0}" rpy="0 0 0"/>
-                </collision>
-                <xacro:cylinder_inertia m="${lidar_mass}" r="${lidar_radius}" h="${lidar_length}"
-                                        xyz="0 0 ${(lidar_length + roof_height)/2.0}" rpy="0 0 0"/>
-            </link>
-            <joint name="base_lidar_joint" type="fixed">
-                <parent link="base_link"/>
-                <child link="lidar_link"/>
-                <origin xyz="0 0 ${S1 + (b + 2*r_caster - S1)}" rpy="0 0 0"/>
-            </joint>
-            <gazebo reference="lidar_link">
-                <material>Gazebo/Black</material>
+                <material>Gazebo/Red</material>
             </gazebo>
         <!-- Wheels -->

File: src/my_amr_description/urdf/my_amr.urdf.xacro (robot description, xacro)
@@ -3,4 +3,5 @@
     <xacro:include filename="common_properties.xacro"/>
     <xacro:include filename="mobile_base.xacro"/>
+    <xacro:include filename="lidar.xacro"/>
     <xacro:include filename="mobile_base_gazebo.xacro"/>
 </robot>
